File: emonTH/board/emonthKsm_1.sch (EAGLE design)
At the start: 9 parts

Commit message: Replaced smd components with regular
Parts:
- C1: device resistor:C-EUC0603 -> rcl:C-EU050-050X075
- R1, R5: device resistor:R-EU_R0603 -> rcl:R-EU_0204/7
- R4: value (none) -> 10k; device resistor:R-EU_R0603 -> rcl:R-EU_0204/7
Connections:
- net 3.3V: now also C1.1
Changed lines of the file:
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@@
 <part name="SUPPLY4" library="supply2" deviceset="GND" device=""/>
 <part name="AMS2302" library="RHT03_DHT-22_AM2302" deviceset="RHT03_DHT-22_AM2302" device=""/>
-<part name="C1" library="resistor" deviceset="C-EU" device="C0603" value="100nf"/>
-<part name="R4" library="resistor" deviceset="R-EU_" device="R0603"/>
-<part name="R5" library="resistor" deviceset="R-EU_" device="R0603" value="4.7k"/>
+<part name="C1" library="rcl" deviceset="C-EU" device="050-050X075" value="100nf"/>
+<part name="R4" library="rcl" deviceset="R-EU_" device="0204/7" value="10k"/>
+<part name="R5" library="rcl" deviceset="R-EU_" device="0204/7" value="4.7k"/>
 <part name="SUPPLY5" library="SparkFun-Aesthetics" deviceset="3.3V" device=""/>
 <part name="SUPPLY6" library="SparkFun-Aesthetics" deviceset="3.3V" device=""/>
-<part name="R1" library="resistor" deviceset="R-EU_" device="R0603" value="100k"/>
+<part name="R1" library="rcl" deviceset="R-EU_" device="0204/7" value="100k"/>
 <part name="SUPPLY9" library="supply2" deviceset="GND" device=""/>
 <part name="SUPPLY10" library="supply2" deviceset="GND" device=""/>
@@
 <pinref part="SUPPLY2" gate="GND" pin="GND"/>
 <pinref part="C1" gate="G$1" pin="2"/>
-<wire x1="172.72" y1="25.4" x2="172.72" y2="22.86" width="0.1524" layer="91"/>
-<wire x1="172.72" y1="22.86" x2="129.54" y2="22.86" width="0.1524" layer="91"/>
+<wire x1="129.54" y1="22.86" x2="172.72" y2="22.86" width="0.1524" layer="91"/>
+<wire x1="172.72" y1="22.86" x2="172.72" y2="25.4" width="0.1524" layer="91"/>
 </segment>
 <segment>
@@
 <wire x1="132.08" y1="66.04" x2="132.08" y2="68.58" width="0.1524" layer="91"/>
 <junction x="132.08" y="68.58"/>
-<wire x1="132.08" y1="68.58" x2="172.72" y2="68.58" width="0.1524" layer="91"/>
-<wire x1="172.72" y1="68.58" x2="172.72" y2="30.48" width="0.1524" layer="91"/>
 <pinref part="SUPPLY5" gate="G$1" pin="3.3V"/>
 <wire x1="132.08" y1="78.74" x2="132.08" y2="68.58" width="0.1524" layer="91"/>
 <pinref part="R1" gate="G$1" pin="2"/>
 <wire x1="127" y1="68.58" x2="132.08" y2="68.58" width="0.1524" layer="91"/>
+<pinref part="C1" gate="G$1" pin="1"/>
+<wire x1="132.08" y1="68.58" x2="172.72" y2="68.58" width="0.1524" layer="91"/>
+<wire x1="172.72" y1="68.58" x2="172.72" y2="33.02" width="0.1524" layer="91"/>
 </segment>
 <segment>

Commit message: Update emonthKSM board
Parts:
- added FRAME1: FRAME-LETTERNO_PACKAGE, SparkFun-Aesthetics:FRAME-LETTERNO_PACKAGE
Other:
- moved on the sheet: AMS2302, ANT1, C1, DS18B20, R1, R4, R5
